File: Toblerone.kicad_pcb (KiCad board)
At the start: 2 copper layers, 342.9 x 142.9 mm, 202 parts, among them J1 Conn_01x04_Pin, K1 KEYSW, K10 KEYSW, K11 KEYSW, K12 KEYSW, K13 KEYSW, K14 KEYSW, K15 KEYSW, K16 KEYSW, K17 KEYSW, K18 KEYSW, K19 KEYSW, K2 KEYSW, K20 KEYSW, K21 KEYSW, K22 KEYSW, K23 KEYSW, K24 KEYSW, K25 KEYSW, K26 KEYSW, K27 KEYSW, K28 KEYSW, K29 KEYSW, K3 KEYSW, K30 KEYSW, K31 KEYSW, K32 KEYSW, K33 KEYSW, K34 KEYSW, K35 KEYSW, K36 KEYSW, K37 KEYSW, K38 KEYSW, K39 KEYSW, K4 KEYSW, K40 KEYSW, K41 KEYSW, K42 KEYSW, K43 KEYSW, K44 KEYSW, K45 KEYSW, K46 KEYSW, K47 KEYSW, K48 KEYSW, K49 KEYSW, K5 KEYSW, K50 KEYSW, K51 KEYSW, K52 KEYSW, K53 KEYSW, K54 KEYSW, K55 KEYSW, K56 KEYSW, K57 KEYSW, K58 KEYSW, K59 KEYSW, K6 KEYSW, K60 KEYSW, K61 KEYSW, K62 KEYSW, K63 KEYSW, K64 KEYSW, K65 KEYSW, K66 KEYSW, K67 KEYSW, K68 KEYSW, K69 KEYSW, K7 KEYSW, K70 KEYSW, K71 KEYSW, K72 KEYSW, K73 KEYSW, K74 KEYSW, K75 KEYSW, K76 KEYSW, K77 KEYSW, K78 KEYSW, K79 KEYSW, K8 KEYSW, K80 KEYSW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

Commit message: PCB design is complete
Parts:
- removed P1: USB_C_Plug_USB2.0, Connector_USB:USB_C_Receptacle_GCT_USB4105-xx-A_16P_TopMnt_Horizontal
- removed X1: XTAL_GND, Crystal:Crystal_SMD_SeikoEpson_FA238-4Pin_3.2x2.5mm
- added G***: LOGO, toblerone-kb_Github_QRCode, F.Cu at (37.4, 39.3)
- added J3: USB_C_Receptacle_USB2.0_14P, Connector_USB:USB_C_Receptacle_GCT_USB4105-xx-A_16P_TopMnt_Horizontal, F.Cu at (56.2, 36.0)
- added Y1: Crystal_GND24, Crystal:Crystal_SMD_SeikoEpson_FA238-4Pin_3.2x2.5mm, F.Cu at (70.8, 47.5)
- D1, D2: footprint Diode_SMD:D_0603_1608Metric -> TobleroneComponets:DIO_LL4148
- D10, D11, D12, D13, D14, D15, D16, D17, D18, D19, D20, D21, D22, D23, D24, D25, D26, D27, D28, D29, D3, D30, D31, D32, D33, D34, D35, D36, D37, D38, D39, D4, D40, D41, D42, D43, D44, D45, D46, D47, D48, D49, D5, D50, D51, D52, D53, D54, D55, D56, D57, D58, D59, D6, D60, D61, D62, D63, D64, D65, D66, D67, D68, D69, D7, D70, D71, D72, D73, D74, D75, D76, D77, D78, D79, D8, D80, D81, D82, D83, D84, D85, D86, D87, D88, D89, D9: footprint Diode_SMD:D_0603_1608Metric -> Diode_SMD:D_MiniMELF
- J1: footprint Connector_PinHeader_1.00mm:PinHeader_1x05_P1.00mm_Horizontal -> TobleroneComponets:AMPHENOL_861400041LO1705LF; moved to B.Cu
- moved C1 7.34 mm to (73.0, 50.4), turned to 90 degrees
- moved C2 7.21 mm to (73.0, 44.0), turned to -90 degrees
- moved R3 3.96 mm to (64.4, 39.7)
- moved R4 3.61 mm to (64.4, 41.2)
- moved C6 2.62 mm to (74.7, 39.9), turned to 90 degrees
- moved J1 2.36 mm to (357.5, 145.1), turned to -90 degrees
- moved C4 1.83 mm to (90.5, 43.0)
- moved C3 1.24 mm to (90.9, 52.9)
- moved D29 0.67 mm to (329.0, 92.8)
- moved C5 0.59 mm to (78.3, 56.1)
- moved C8 0.55 mm to (81.6, 38.9)
- moved C7 0.41 mm to (86.8, 39.0)
- moved D62 0.32 mm to (329.0, 130.5)
- moved S1 0.22 mm to (281.1, 145.7)
- moved S3 0.21 mm to (128.7, 164.8)
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Connections:
- net Col1 renamed /Col1
- net Col2 renamed /Col2
- net Col3 renamed /Col3
- net Col4 renamed /Col4
- net Col5 renamed /Col5
- net Col6 renamed /Col6
- C1 pad 1: Net-(U1-XTAL2) -> GND
- C1 pad 2: GND -> Net-(U1-XTAL1)
- C2 pad 1: Net-(U1-XTAL1) -> GND
- C2 pad 2: GND -> Net-(U1-XTAL2)
- D10 pad 1: Row1 -> /Row1
- D11 pad 1: Row1 -> /Row1
- D12 pad 1: Row1 -> /Row1
- D13 pad 1: Row1 -> /Row1
- D14 pad 1: Row1 -> /Row1
- D15 pad 1: Row2 -> /Row2
- D16 pad 1: Row2 -> /Row2
- D17 pad 1: Row2 -> /Row2
- D18 pad 1: Row2 -> /Row2
- D19 pad 1: Row2 -> /Row2
- D20 pad 1: Row2 -> /Row2
- D21 pad 1: Row2 -> /Row2
- D22 pad 1: Row2 -> /Row2
- D23 pad 1: Row2 -> /Row2
- D24 pad 1: Row2 -> /Row2
- D25 pad 1: Row2 -> /Row2
- D26 pad 1: Row2 -> /Row2
- D27 pad 1: Row2 -> /Row2
- D28 pad 1: Row2 -> /Row2
- D29 pad 1: Row2 -> /Row1
- D3 pad 1: Row1 -> /Row1
- D30 pad 1: Row2 -> /Row1
- D31 pad 1: Row2 -> /Row6
- D32 pad 1: Row3 -> /Row3
- D33 pad 1: Row3 -> /Row3
- D34 pad 1: Row3 -> /Row3
- D35 pad 1: Row3 -> /Row3
- D36 pad 1: Row3 -> /Row3
- D37 pad 1: Row3 -> /Row3
- D38 pad 1: Row3 -> /Row3
- D39 pad 1: Row3 -> /Row3
- D4 pad 1: Row1 -> /Row1
- D40 pad 1: Row3 -> /Row3
- D41 pad 1: Row3 -> /Row3
- D42 pad 1: Row3 -> /Row3
- D43 pad 1: Row3 -> /Row3
- D44 pad 1: Row3 -> /Row3
- D45 pad 1: Row3 -> /Row3
- D46 pad 1: Row3 -> /Row2
- D47 pad 1: Row3 -> /Row2
- D48 pad 1: Row3 -> /Row5
- D49 pad 1: Row4 -> /Row4
- D5 pad 1: Row1 -> /Row1
- D50 pad 1: Row4 -> /Row4
- D51 pad 1: Row4 -> /Row4
- D52 pad 1: Row4 -> /Row4
- D53 pad 1: Row4 -> /Row4
- D54 pad 1: Row4 -> /Row4
- D55 pad 1: Row4 -> /Row4
- D56 pad 1: Row4 -> /Row4
- D57 pad 1: Row4 -> /Row4
- D58 pad 1: Row4 -> /Row4
- D59 pad 1: Row4 -> /Row4
- D6 pad 1: Row1 -> /Row1
- D60 pad 1: Row4 -> /Row4
- D61 pad 1: Row4 -> /Row4
- D62 pad 1: Row4 -> /Row3
- D63 pad 1: Row4 -> /Row3
- D64 pad 1: Row4 -> /Row4
- D65 pad 1: Row5 -> /Row5
- D66 pad 1: Row5 -> /Row5
- D67 pad 1: Row5 -> /Row5
- D68 pad 1: Row5 -> /Row5
- D69 pad 1: Row5 -> /Row5
- D7 pad 1: Row1 -> /Row1
- D70 pad 1: Row5 -> /Row5
- D71 pad 1: Row5 -> /Row5
- D72 pad 1: Row5 -> /Row5
- D73 pad 1: Row5 -> /Row5
- D74 pad 1: Row5 -> /Row5
- D75 pad 1: Row5 -> /Row5
- D76 pad 1: Row5 -> /Row5
- D77 pad 1: Row5 -> /Row5
- D78 pad 1: Row6 -> /Row6
- D79 pad 1: Row6 -> /Row6
- D8 pad 1: Row1 -> /Row1
- D80 pad 1: Row6 -> /Row6
- D81 pad 1: Row6 -> /Row6
- D82 pad 1: Row6 -> /Row6
- D83 pad 1: Row6 -> /Row6
- D84 pad 1: Row6 -> /Row6
- D85 pad 1: Row6 -> /Row6
- D86 pad 1: Row6 -> /Row6
- D87 pad 1: Row6 -> /Row6
- D88 pad 1: Row6 -> /Row6
- D89 pad 1: Row6 -> /Row5
- D9 pad 1: Row1 -> /Row1
- D90 pad 2: Net-(U1-AREF) -> /capslock
- K10 pad 1: Col10 -> /Col10
- K11 pad 1: Col11 -> /Col11
- K12 pad 1: Col12 -> /Col12
- K13 pad 1: Col13 -> /Col13
- K14 pad 1: Col14 -> /Col14
- K21 pad 1: Col7 -> /Col7
- K22 pad 1: Col8 -> /Col8
- K23 pad 1: Col9 -> /Col9
- K24 pad 1: Col10 -> /Col10
- K25 pad 1: Col11 -> /Col11
- K26 pad 1: Col12 -> /Col12
- K27 pad 1: Col13 -> /Col13
- K28 pad 1: Col14 -> /Col14
- K29 pad 1: Col15 -> /Col15
- K30 pad 1: Col16 -> /Col16
- K31 pad 1: Col17 -> /Col16
- K38 pad 1: Col7 -> /Col7
- K39 pad 1: Col8 -> /Col8
- K40 pad 1: Col9 -> /Col9
- K41 pad 1: Col10 -> /Col10
- K42 pad 1: Col11 -> /Col11
- K43 pad 1: Col12 -> /Col12
- K44 pad 1: Col13 -> /Col13
- K45 pad 1: Col14 -> /Col14
- K46 pad 1: Col15 -> /Col15
- K47 pad 1: Col16 -> /Col16
- K48 pad 1: Col17 -> /Col16
- K55 pad 1: Col7 -> /Col7
- K56 pad 1: Col8 -> /Col8
- K57 pad 1: Col9 -> /Col9
- K58 pad 1: Col10 -> /Col10
- K59 pad 1: Col11 -> /Col11
- K60 pad 1: Col12 -> /Col12
- K61 pad 1: Col13 -> /Col13
- K62 pad 1: Col15 -> /Col15
- K63 pad 1: Col16 -> /Col16
- K64 pad 1: Col17 -> /Col16
- K7 pad 1: Col7 -> /Col7
- K71 pad 1: Col7 -> /Col7
- K72 pad 1: Col8 -> /Col8
- K73 pad 1: Col9 -> /Col9
- K74 pad 1: Col10 -> /Col10
- K75 pad 1: Col11 -> /Col11
- K76 pad 1: Col12 -> /Col13
- K77 pad 1: Col16 -> /Col14
- K8 pad 1: Col8 -> /Col8
- K82 pad 1: Col7 -> /Col8
- K83 pad 1: Col8 -> /Col10
- K84 pad 1: Col9 -> /Col11
- K85 pad 1: Col10 -> /Col12
- K86 pad 1: Col11 -> /Col13
- K87 pad 1: Col15 -> /Col14
- K88 pad 1: Col16 -> /Col15
- K89 pad 1: Col17 -> /Col15
- K9 pad 1: Col9 -> /Col9
- U1 pad 1: Row6 -> /Row6
- U1 pad 10: Row3 -> /Row3
- U1 pad 11: Row2 -> /Row2
- U1 pad 12: Row1 -> /Row1
- U1 pad 26: Col7 -> /Col7
- U1 pad 27: Col8 -> /Col8
- U1 pad 28: Col9 -> /Col9
- U1 pad 29: Col10 -> /Col10
- U1 pad 30: Col11 -> /Col11
- U1 pad 31: Col12 -> /Col12
- U1 pad 32: Col13 -> /Col13
- U1 pad 38: Col14 -> /Col14
- U1 pad 39: Col15 -> /Col15
- U1 pad 40: Col16 -> /Col16
- U1 pad 41: Col17 -> /capslock
- U1 pad 42: Net-(U1-AREF) -> unconnected-(U1-AREF-Pad42)
- U1 pad 7: Net-(U1-VBUS) -> VCC
- U1 pad 8: Row5 -> /Row5
- U1 pad 9: Row4 -> /Row4
Routing:
- net /Row6: track 0.00 -> 596.7 mm, vias 0 -> 1
- net /Row5: track 0.00 -> 552.6 mm, vias 0 -> 1
- net Row6: track 509.7 -> 0.00 mm, vias 1 -> 0
- net /Row4: track 0.00 -> 467.9 mm, vias 0 -> 1
- net Row5: track 463.0 -> 0.00 mm, vias 1 -> 0
- net Row4: track 460.9 -> 0.00 mm, vias 1 -> 0
- net Row3: track 444.0 -> 0.00 mm, vias 1 -> 0
- net Row2: track 440.6 -> 0.00 mm, vias 1 -> 0
- net /Row3: track 0.00 -> 435.6 mm, vias 0 -> 3
- net /Row1: track 0.00 -> 424.0 mm, vias 0 -> 1
- net /Row2: track 0.00 -> 419.4 mm, vias 0 -> 1
- net /Col16: track 0.00 -> 374.6 mm, vias 0 -> 3
- net Col17: track 374.3 -> 0.00 mm, vias 3 -> 0
- net /Col14: track 0.00 -> 371.4 mm, vias 0 -> 4
- net /Col15: track 0.00 -> 367.2 mm, vias 0 -> 3
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Other:
- board text added: "KingCast Designs 2025 Board Rev: 031"
- board text added: "R1C1"
- board text added: "R1C10"
- board text added: "R1C11"
- board text added: "R1C12"
- board text added: "R1C13"
- board text added: "R1C14"
- board text added: "R1C15"
- board text added: "R1C16"
- board text added: "R1C2"
- board text added: "R1C3"
- board text added: "R1C4"
- board text added: "R1C5"
- board text added: "R1C6"
- board text added: "R1C7"
- board text added: "R1C8"
- board text added: "R1C9"
- board text added: "R2C1"
- board text added: "R2C10"
- board text added: "R2C11"
- board text added: "R2C12"
- board text added: "R2C13"
- board text added: "R2C14"
- board text added: "R2C15"
- board text added: "R2C16"
- board text added: "R2C2"
- board text added: "R2C3"
- board text added: "R2C4"
- board text added: "R2C5"
- board text added: "R2C6"
- board text added: "R2C7"
- board text added: "R2C8"
- board text added: "R2C9"
- board text added: "R3C1"
- board text added: "R3C10"
- board text added: "R3C11"
- board text added: "R3C12"
- board text added: "R3C13"
- board text added: "R3C14"
- board text added: "R3C15"
- board text added: "R3C16"
- board text added: "R3C2"
- board text added: "R3C3"
- board text added: "R3C4"
- board text added: "R3C5"
- board text added: "R3C6"
- board text added: "R3C7"
- board text added: "R3C8"
- board text added: "R3C9"
- board text added: "R4C1"
- board text added: "R4C10"
- board text added: "R4C11"
- board text added: "R4C12"
- board text added: "R4C13"
- board text added: "R4C16"
- board text added: "R4C2"
- board text added: "R4C3"
- board text added: "R4C4"
- board text added: "R4C5"
- board text added: "R4C6"
- board text added: "R4C7"
- board text added: "R4C8"
- board text added: "R4C9"
- board text added: "R5C1"
- board text added: "R5C10"
- board text added: "R5C11"
- board text added: "R5C13"
- board text added: "R5C14"
- board text added: "R5C15"
- board text added: "R5C16"
- board text added: "R5C2"
- board text added: "R5C3"
- board text added: "R5C4"
- board text added: "R5C5"
- board text added: "R5C6"
- board text added: "R5C7"
- board text added: "R5C8"
- board text added: "R5C9"
- board text added: "R6C1"
- board text added: "R6C10"
- board text added: "R6C11"
- board text added: "R6C12"
- board text added: "R6C13"
- board text added: "R6C14"
- board text added: "R6C15"
- board text added: "R6C16"
- board text added: "R6C2"
- board text added: "R6C3"
- board text added: "R6C5"
- board text added: "R6C8"
- board text added: "Toblerone Keyboard"
- board text added: "USB-C"
