File: Toblerone.kicad_sch (KiCad schematic)
At the start: 206 parts, among them J1 Conn_01x04_Pin, J2 Conn_01x04_Socket, K1 KEYSW, K10 KEYSW, K11 KEYSW, K12 KEYSW, K13 KEYSW, K14 KEYSW, K15 KEYSW, K16 KEYSW, K17 KEYSW, K18 KEYSW, K19 KEYSW, K2 KEYSW, K20 KEYSW, K21 KEYSW, K22 KEYSW, K23 KEYSW, K24 KEYSW, K25 KEYSW, K26 KEYSW, K27 KEYSW, K28 KEYSW, K29 KEYSW, K3 KEYSW, K30 KEYSW, K31 KEYSW, K32 KEYSW, K33 KEYSW, K34 KEYSW, K35 KEYSW, K36 KEYSW, K37 KEYSW, K38 KEYSW, K39 KEYSW, K4 KEYSW, K40 KEYSW, K41 KEYSW, K42 KEYSW, K43 KEYSW, K44 KEYSW, K45 KEYSW, K46 KEYSW, K47 KEYSW, K48 KEYSW, K49 KEYSW, K5 KEYSW, K50 KEYSW, K51 KEYSW, K52 KEYSW, K53 KEYSW, K54 KEYSW, K55 KEYSW, K56 KEYSW, K57 KEYSW, K58 KEYSW, K59 KEYSW, K6 KEYSW, K60 KEYSW, K61 KEYSW, K62 KEYSW, K63 KEYSW, K64 KEYSW, K65 KEYSW, K66 KEYSW, K67 KEYSW, K68 KEYSW, K69 KEYSW, K7 KEYSW, K70 KEYSW, K71 KEYSW, K72 KEYSW, K73 KEYSW, K74 KEYSW, K75 KEYSW, K76 KEYSW, K77 KEYSW, K78 KEYSW, K79 KEYSW, K8 KEYSW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

Commit message: PCB design is complete
Parts:
- removed P1: USB_C_Plug_USB2.0, Connector_USB:USB_C_Receptacle_GCT_USB4105-xx-A_16P_TopMnt_Horizontal, symbol Connector:USB_C_Plug_USB2.0
- removed X1: XTAL_GND, Crystal:Crystal_SMD_SeikoEpson_FA238-4Pin_3.2x2.5mm, symbol keyboard_parts:XTAL_GND
- added J3: USB_C_Receptacle_USB2.0_14P, Connector_USB:USB_C_Receptacle_GCT_USB4105-xx-A_16P_TopMnt_Horizontal, symbol Connector:USB_C_Receptacle_USB2.0_14P
- added Y1: Crystal_GND24, Crystal:Crystal_SMD_SeikoEpson_FA238-4Pin_3.2x2.5mm, symbol Device:Crystal_GND24
- D1, D2: footprint Diode_SMD:D_0603_1608Metric -> TobleroneComponets:DIO_LL4148; symbol Device:D -> Diode:LL4148
- D10, D11, D12, D13, D14, D15, D16, D17, D18, D19, D20, D21, D22, D23, D24, D25, D26, D27, D28, D29, D3, D30, D31, D32, D33, D34, D35, D36, D37, D38, D39, D4, D40, D41, D42, D43, D44, D45, D46, D47, D48, D49, D5, D50, D51, D52, D53, D54, D55, D56, D57, D58, D59, D6, D60, D61, D62, D63, D64, D65, D66, D67, D68, D69, D7, D70, D71, D72, D73, D74, D75, D76, D77, D78, D79, D8, D80, D81, D82, D83, D84, D85, D86, D87, D88, D89, D9: footprint Diode_SMD:D_0603_1608Metric -> Diode_SMD:D_MiniMELF; symbol Device:D -> Diode:LL4148
- J1: footprint Connector_PinHeader_1.00mm:PinHeader_1x05_P1.00mm_Horizontal -> TobleroneComponets:AMPHENOL_861400041LO1705LF
Connections:
- net Col10: now also K83.1; no longer K85.1
- net Col11: now also K84.1; no longer K86.1
- net Col12: now also K85.1; no longer K76.1
- net Col13: now also K76.1, K86.1
- net Col14: now also K77.1, K87.1
- net Col15: now also K88.1, K89.1; no longer K87.1
- net Col16: now also K31.1, K48.1, K64.1; no longer K77.1, K88.1
- net Col7: no longer K82.1
- net Col8: now also K82.1; no longer K83.1
- net Col9: no longer K84.1
- net GND: now also C1.1, C2.1, J3.A1 (GND), J3.A12 (GND), J3.B1 (GND), J3.B12 (GND), J3.S1 (SHIELD), Y1.2, Y1.4; no longer C1.2, C2.2
- net Row1: now also D29.1 (K), D30.1 (K)
- net Row2: now also D46.1 (K), D47.1 (K); no longer D29.1 (K), D30.1 (K), D31.1 (K)
- net Row3: now also D62.1 (K), D63.1 (K); no longer D46.1 (K), D47.1 (K), D48.1 (K)
- net Row4: no longer D62.1 (K), D63.1 (K)
- net Row5: now also D48.1 (K), D89.1 (K)
- net Row6: now also D31.1 (K); no longer D89.1 (K)
- net VCC: now also U1.7 (VBUS), J3.A4 (VBUS), J3.A9 (VBUS), J3.B4 (VBUS), J3.B9 (VBUS)
- net at U1.17 (XTAL1): now also C1.2, Y1.1; no longer C2.1
- net at U1.16 (XTAL2): now also C2.2, Y1.3; no longer C1.1
- net at R4.2: now also J3.A6 (D+), J3.B6 (D+)
- net at R3.2: now also J3.A7 (D-), J3.B7 (D-)
- net at U1.42 (AREF): no longer D90.2
- removed net Col17: K31.1, K48.1, K64.1, K89.1, U1.41 (PF0)
- new net capslock: D90.2, U1.41 (PF0)
- no-connect marks 0 -> 2
Other:
- moved on the sheet: C1, C2, C8, D29, D30, D31, D46, D47, D48, D62, D63, D64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
